File: cw308_fe310.kicad_pcb (KiCad board)
At the start: 2 copper layers, 28 parts, among them J1 CW308T_CONNBOARD, J2 Conn_02x02_Odd_Even, SW1 SW_Push, U1 IS25LP128, U2 SN74LVC1G04DBVR, U3 FE310-G000, U4 SN74LVC1G07DBVR, U5 SN74LVC1G07DBVR, Y1 16Mhz

Commit message: progress
Parts:
- removed 100R1: R, Resistor_SMD:R_0603_1608Metric_Pad1.05x0.95mm_HandSolder
- added C14: 0.1uF, Capacitor_SMD:C_0603_1608Metric_Pad1.05x0.95mm_HandSolder, F.Cu at (76.5, 34.4)
- added C15: 4.7uF, Capacitor_SMD:C_0603_1608Metric_Pad1.05x0.95mm_HandSolder, F.Cu at (70.8, 37.5)
- added C16: 4.7uF, Capacitor_SMD:C_0603_1608Metric_Pad1.05x0.95mm_HandSolder, F.Cu at (64.8, 39.3)
- added C17: 0.1uF, Capacitor_SMD:C_0603_1608Metric_Pad1.05x0.95mm_HandSolder, F.Cu at (79.4, 28.0)
- added C18: 0.1uF, Capacitor_SMD:C_0603_1608Metric_Pad1.05x0.95mm_HandSolder, F.Cu at (76.5, 32.9)
- added C19: 4.7uF, Capacitor_SMD:C_0603_1608Metric_Pad1.05x0.95mm_HandSolder, F.Cu at (82.7, 29.5)
- added C20: 12pF, Capacitor_SMD:C_0603_1608Metric_Pad1.05x0.95mm_HandSolder, F.Cu at (74.8, 40.5)
- added C21: 12pF, Capacitor_SMD:C_0603_1608Metric_Pad1.05x0.95mm_HandSolder, F.Cu at (79.8, 32.5)
- added C22: 0.1uF, Capacitor_SMD:C_0603_1608Metric_Pad1.05x0.95mm_HandSolder, F.Cu at (82.7, 28.0)
- added C23: 0.1uF, Capacitor_SMD:C_0603_1608Metric_Pad1.05x0.95mm_HandSolder, F.Cu at (104.6, 50.8)
- added C24: 0.1uF, Capacitor_SMD:C_0603_1608Metric_Pad1.05x0.95mm_HandSolder, F.Cu at (79.4, 31.0)
- added C25: 0.1uF, Capacitor_SMD:C_0603_1608Metric_Pad1.05x0.95mm_HandSolder, F.Cu at (117.0, 38.6)
- added C26: 0.1uF, Capacitor_SMD:C_0603_1608Metric_Pad1.05x0.95mm_HandSolder, F.Cu at (74.2, 37.5)
- added C27: 0.1uF, Capacitor_SMD:C_0603_1608Metric_Pad1.05x0.95mm_HandSolder, F.Cu at (117.2, 55.1)
- added C28: 0.1uF, Capacitor_SMD:C_0603_1608Metric_Pad1.05x0.95mm_HandSolder, F.Cu at (79.4, 29.5)
- added C29: 0.1uF, Capacitor_SMD:C_0603_1608Metric_Pad1.05x0.95mm_HandSolder, F.Cu at (104.6, 43.2)
- added D1: PGB1010603MR, digikey-footprints:0603, F.Cu at (61.0, 40.8)
- added D2: PGB1010603MR, digikey-footprints:0603, F.Cu at (63.6, 40.8)
- added FB1: MPZ2012S601AT000, digikey-footprints:0805, F.Cu at (57.8, 39.5)
- added FB2: MPZ2012S601AT000, digikey-footprints:0805, F.Cu at (79.6, 26.3)
- added J3: 10118193-0001LF, digikey-footprints:USB_Micro_B_Female_10118193-0001LF, F.Cu at (114.3, 29.2)
- added JP1: Jumper, Connector_PinHeader_2.54mm:PinHeader_1x02_P2.54mm_Vertical, F.Cu at (150.5, 51.7)
- added JP2: Clock_Src_Sel, Connector_PinHeader_2.54mm:PinHeader_1x03_P2.54mm_Vertical, F.Cu at (160.1, 38.7)
- added JP5: TDI_SEL, Connector_PinHeader_2.54mm:PinHeader_1x03_P2.54mm_Vertical, F.Cu at (231.0, 38.7)
- added JP6: TX_SEL, Connector_PinHeader_2.54mm:PinHeader_1x03_P2.54mm_Vertical, F.Cu at (220.0, 38.7)
- added JP7: RX_SEL, Connector_PinHeader_2.54mm:PinHeader_1x03_P2.54mm_Vertical, F.Cu at (241.9, 38.7)
- added JP8: TDO_SEL, Connector_PinHeader_2.54mm:PinHeader_1x03_P2.54mm_Vertical, F.Cu at (238.3, 38.7)
- added JP9: TCK_SEL, Connector_PinHeader_2.54mm:PinHeader_1x03_P2.54mm_Vertical, F.Cu at (234.6, 38.7)
- added R10: 1K, Resistor_SMD:R_0603_1608Metric_Pad1.05x0.95mm_HandSolder, F.Cu at (76.5, 35.9)
- added R4: 100, Resistor_SMD:R_0603_1608Metric_Pad1.05x0.95mm_HandSolder, F.Cu at (167.0, 43.5)
- added R5: 1K, Resistor_SMD:R_0603_1608Metric_Pad1.05x0.95mm_HandSolder, F.Cu at (74.8, 39.0)
- added R6: 1K, Resistor_SMD:R_0603_1608Metric_Pad1.05x0.95mm_HandSolder, F.Cu at (79.8, 34.0)
- added R7: 12K, Resistor_SMD:R_0603_1608Metric_Pad1.05x0.95mm_HandSolder, F.Cu at (82.7, 31.0)
- added R8: 1K, Resistor_SMD:R_0603_1608Metric_Pad1.05x0.95mm_HandSolder, F.Cu at (77.5, 37.4)
- added R9: 1K, Resistor_SMD:R_0603_1608Metric_Pad1.05x0.95mm_HandSolder, F.Cu at (71.5, 40.5)
- added TP1: TestPoint, TestPoint:TestPoint_Pad_D1.5mm, F.Cu at (172.1, 38.1)
- added TP2: TestPoint, TestPoint:TestPoint_Pad_D1.5mm, F.Cu at (153.7, 57.9)
- added TP3: TestPoint, TestPoint:TestPoint_Pad_D1.5mm, F.Cu at (150.0, 61.6)
- added Y2: 12MHz, Crystal:Crystal_SMD_TXC_7M-4Pin_3.2x2.5mm_HandSoldering, F.Cu at (72.0, 34.4)
- C11, C12: value 12pF -> 0.1uF
- C2: value 0.1uF -> 12pF
- C3: value 100n -> 12pF
- C4: value 10nF -> 0.1uF
- C5: value 10uF -> 0.1uF
- C6: value 0.1uF -> 100n
- C7: value 0.1uF -> 10nF
- J2: value Conn_02x02_Odd_Even -> CrystalJumper; footprint Connector_PinHeader_2.54mm:PinHeader_2x02_P2.54mm_Vertical_SMD -> Connector_PinHeader_2.54mm:PinHeader_2x02_P2.54mm_Vertical
- JP3: value Jumper -> TMS_SEL; footprint Connector_PinHeader_2.54mm:PinHeader_1x02_P2.54mm_Vertical_SMD_Pin1Left -> Connector_PinHeader_2.54mm:PinHeader_1x03_P2.54mm_Vertical
- JP4: value Clock_Src_Sel -> RST_SEL; footprint Connector_PinHeader_2.54mm:PinHeader_1x03_P2.54mm_Vertical_SMD_Pin1Left -> Connector_PinHeader_2.54mm:PinHeader_1x03_P2.54mm_Vertical
- U2: value SN74LVC1G04DBVR -> SN74LVC1G07DBVR
- U3: value FE310-G000 -> SN74LVC1G07DBVR; footprint Package_DFN_QFN:QFN-48-1EP_6x6mm_P0.4mm_EP4.66x4.66mm_ThermalVias -> digikey-footprints:SOT-753
- U4: value SN74LVC1G07DBVR -> FE310-G000; footprint digikey-footprints:SOT-753 -> Package_DFN_QFN:QFN-48-1EP_6x6mm_P0.4mm_EP4.66x4.66mm_ThermalVias
- U5: value SN74LVC1G07DBVR -> FT2232HL-REEL; footprint digikey-footprints:SOT-753 -> digikey-footprints:LQFP-64_10x10mm
- moved C11 148.2 mm to (57.6, 21.4)
- moved R2 141.4 mm to (67.6, 21.4)
- moved C3 138.5 mm to (57.6, 19.9)
- moved C10 132.4 mm to (60.9, 19.9)
- moved C5 128.0 mm to (64.3, 21.4)
- moved C6 127.3 mm to (64.3, 19.9)
- moved C8 126.0 mm to (60.9, 21.4)
- moved C1 124.9 mm to (67.6, 19.9)
- moved C4 90.4 mm to (166.9, 42.0)
- moved U5 85.8 mm to (114.3, 47.0)
- moved SW1 77.5 mm to (154.8, 53.4)
- moved U4 72.7 mm to (114.3, 73.7)
- moved U3 55.4 mm to (169.0, 39.0)
- moved U2 51.9 mm to (150.6, 58.2)
- moved J1 48.7 mm to (90.2, 38.1)
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Connections:
- net +1V2 renamed Net-(J1-PadC11)
- net +2V5 renamed Net-(J1-PadC13)
- net +5V renamed Net-(J1-PadC15)
- C10 pad 1: Net-(100R1-Pad2) -> +3V3
- C10 pad 2: PLL_AVSS -> GND
- C11 pad 1: Net-(C11-Pad1) -> GND
- C11 pad 2: Net-(C11-Pad2) -> +1V8
- C12 pad 2: Net-(C12-Pad2) -> PLL_AVSS
- C13 pad 1: +1V8 -> Net-(C12-Pad1)
- C13 pad 2: GND -> PLL_AVSS
- C2 pad 1: +1V8 -> Net-(C2-Pad1)
- C2 pad 2: GND -> Net-(C2-Pad2)
- C3 pad 1: GND -> Net-(C3-Pad1)
- C4 pad 1: Net-(C4-Pad1) -> +1V8
- C5 pad 1: +3V3 -> +1V8
- C6 pad 1: +3V3 -> GND
- C6 pad 2: GND -> Net-(C6-Pad2)
- C7 pad 1: +3V3 -> Net-(C7-Pad1)
- C8 pad 1: GND -> +3V3
- C8 pad 2: +1V8 -> GND
- C9 pad 1: Net-(100R1-Pad2) -> +3V3
- C9 pad 2: PLL_AVSS -> GND
- J1 pad A11: RST -> UFO.RST
- J1 pad B2: JTAG_TRST -> UFO.JTAG_TRST
- J1 pad B3: JTAG_TDI -> UFO.JTAG_TDI
- J1 pad B4: JTAG_TDO -> UFO.JTAG_TDO
- J1 pad B5: JTAG_TMS -> UFO.JTAG_TMS
- J1 pad B6: JTAG_TCK -> UFO.JTAG_TCK
- J1 pad C3: Net-(C3-Pad2) -> Net-(C6-Pad2)
- J1 pad C5: Net-(C3-Pad2) -> Net-(C6-Pad2)
- J2 pad 1: Net-(C11-Pad1) -> Net-(C2-Pad1)
- J2 pad 3: Net-(C12-Pad1) -> Net-(C3-Pad1)
- JP3 pad 1: CLKOUT -> FTDI.JTAG_TMS
- JP3 pad 2: XTAL_XO -> JTAG_TMS
- JP4 pad 1: CLKIN -> FTDI.RESET
- JP4 pad 2: XTAL_XI -> JTAG_RESET
- JP4 pad 3: Net-(J2-Pad2) -> UFO.JTAG_TRST
- R1 pad 2: Net-(C3-Pad2) -> Net-(C6-Pad2)
- R2 pad 2: Net-(C4-Pad1) -> Net-(C7-Pad1)
- SW1 pad 2: Net-(C4-Pad1) -> Net-(C7-Pad1)
- U2 pad 2: JTAG_TRST -> UFO.RST
- U2 pad 4: JTAG_TRST_N -> Net-(C7-Pad1)
- U2 pad 5: +3V3 -> +1V8
- U3 pad 1: FLASH_IO3 -> Net-(U3-Pad1)
- U3 pad 2: FLASH_IO2 -> JTAG_TRST
- U3 pad 3: FLASH_IO1 -> GND
- U3 pad 4: FLASH_IO0 -> Net-(C7-Pad1)
- U3 pad 5: FLASH_S -> +1V8
- U4 pad 1: Net-(U4-Pad1) -> FLASH_IO3
- U4 pad 2: RST -> FLASH_IO2
- U4 pad 3: GND -> FLASH_IO1
- U4 pad 4: Net-(C4-Pad1) -> FLASH_IO0
- U4 pad 5: +1V8 -> FLASH_S
- U5 pad 1: Net-(U5-Pad1) -> GND
- U5 pad 2: JTAG_TRST_N -> Net-(C21-Pad1)
- U5 pad 3: GND -> Net-(C20-Pad1)
- U5 pad 4: Net-(C4-Pad1) -> Net-(C16-Pad1)
- U5 pad 5: +1V8 -> GND
- Y1 pad 1: Net-(C11-Pad1) -> Net-(C2-Pad1)
- Y1 pad 3: Net-(C12-Pad1) -> Net-(C3-Pad1)
Other:
- board outline added: 53.3 x 67.3 mm

Commit message: progress update
Parts:
- removed JP3: TMS_SEL, Connector_PinHeader_2.54mm:PinHeader_1x03_P2.54mm_Vertical
- removed JP4: RST_SEL, Connector_PinHeader_2.54mm:PinHeader_1x03_P2.54mm_Vertical
- removed JP5: TDI_SEL, Connector_PinHeader_2.54mm:PinHeader_1x03_P2.54mm_Vertical
- removed JP8: TDO_SEL, Connector_PinHeader_2.54mm:PinHeader_1x03_P2.54mm_Vertical
- removed JP9: TCK_SEL, Connector_PinHeader_2.54mm:PinHeader_1x03_P2.54mm_Vertical
- added J4: Conn_02x05_Odd_Even, Connector_PinHeader_2.54mm:PinHeader_2x05_P2.54mm_Vertical, F.Cu at (100.1, 65.5)
- moved JP7 117.4 mm to (131.6, 78.7)
- moved JP6 101.0 mm to (127.3, 78.7)
- moved C1 88.8 mm to (125.5, 87.2)
- moved C4 79.1 mm to (102.0, 87.1)
- moved C10 75.0 mm to (114.6, 72.3), turned to 180 degrees
- moved C8 73.9 mm to (120.8, 64.7), turned to 90 degrees
- moved C6 73.8 mm to (132.1, 49.0)
- moved C3 71.3 mm to (126.1, 39.5)
- moved R2 69.2 mm to (112.8, 73.8)
- moved U3 67.1 mm to (107.0, 64.5), turned to 270 degrees
- moved C11 67.0 mm to (111.1, 61.6)
- moved Y1 66.9 mm to (109.7, 77.3)
- moved C5 62.8 mm to (111.0, 63.2), turned to 180 degrees
- moved C12 60.0 mm to (114.3, 76.3)
- moved Y2 59.0 mm to (130.3, 42.9)
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Connections:
- J1 pad B2: UFO.JTAG_TRST -> Net-(J1-PadB2)
- J1 pad B3: UFO.JTAG_TDI -> Net-(J1-PadB3)
- J1 pad B4: UFO.JTAG_TDO -> Net-(J1-PadB4)
- J1 pad B5: UFO.JTAG_TMS -> Net-(J1-PadB5)
- J1 pad B6: UFO.JTAG_TCK -> Net-(J1-PadB6)
Routing:
- net GND: track 0.00 -> 67.5 mm, vias 0 -> 4
- net FTDI.JTAG_TCK: track 0.00 -> 45.4 mm
- net FTDI.JTAG_TDI: track 0.00 -> 38.6 mm
- net FTDI.JTAG_TDO: track 0.00 -> 35.2 mm
- net +1V8: track 0.00 -> 34.2 mm
- net FTDI.JTAG_TMS: track 0.00 -> 32.4 mm
- net JTAG_TCK: track 0.00 -> 27.7 mm, vias 0 -> 1
- net +3V3: track 0.00 -> 23.9 mm
- net JTAG_TDI: track 0.00 -> 23.0 mm, vias 0 -> 2
- net JTAG_TDO: track 0.00 -> 22.8 mm, vias 0 -> 2
- net FTDI.RESET: track 0.00 -> 21.5 mm
- net JTAG_TMS: track 0.00 -> 19.5 mm, vias 0 -> 2
- net DP: track 0.00 -> 18.3 mm
- net FLASH_S: track 0.00 -> 16.4 mm
- net FLASH_IO1: track 0.00 -> 16.3 mm, vias 0 -> 2
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Other:
- net class Default: clearance 0.2 -> 0.127
- rule trace_clearance: 0.2 -> 0.127
- rule trace_min: 0.2 -> 0.0889
- rule via_min_drill: 0.3 -> 0.2
- rule via_min_size: 0.4 -> 0.45

Commit message: simplified prototype ready
Parts:
- removed C14, C17, C18, C22, C23, C24, C25, C26, C27, C28, C29: 0.1uF, Capacitor_SMD:C_0603_1608Metric_Pad1.05x0.95mm_HandSolder
- removed C15, C16, C19: 4.7uF, Capacitor_SMD:C_0603_1608Metric_Pad1.05x0.95mm_HandSolder
- removed C2, C20, C21, C3: 12pF, Capacitor_SMD:C_0603_1608Metric_Pad1.05x0.95mm_HandSolder
- removed D1, D2: PGB1010603MR, digikey-footprints:0603
- removed FB1, FB2: MPZ2012S601AT000, digikey-footprints:0805
- removed J2: CrystalJumper, Connector_PinHeader_2.54mm:PinHeader_2x02_P2.54mm_Vertical
- removed J3: 10118193-0001LF, digikey-footprints:USB_Micro_B_Female_10118193-0001LF
- removed J4: Conn_02x05_Odd_Even, Connector_PinHeader_2.54mm:PinHeader_2x05_P2.54mm_Vertical
- removed JP1: Jumper, Connector_PinHeader_2.54mm:PinHeader_1x02_P2.54mm_Vertical
- removed JP2: Clock_Src_Sel, Connector_PinHeader_2.54mm:PinHeader_1x03_P2.54mm_Vertical
- removed JP6: TX_SEL, Connector_PinHeader_2.54mm:PinHeader_1x03_P2.54mm_Vertical
- removed JP7: RX_SEL, Connector_PinHeader_2.54mm:PinHeader_1x03_P2.54mm_Vertical
- removed R10, R5, R6, R8, R9: 1K, Resistor_SMD:R_0603_1608Metric_Pad1.05x0.95mm_HandSolder
- removed R7: 12K, Resistor_SMD:R_0603_1608Metric_Pad1.05x0.95mm_HandSolder
- removed TP1, TP2, TP3: TestPoint, TestPoint:TestPoint_Pad_D1.5mm
- removed U5: FT2232HL-REEL, digikey-footprints:LQFP-64_10x10mm
- removed Y1: 16Mhz, Oscillator:Oscillator_SMD_Abracon_ASE-4Pin_3.2x2.5mm_HandSoldering
- removed Y2: 12MHz, Crystal:Crystal_SMD_TXC_7M-4Pin_3.2x2.5mm_HandSoldering
- moved C4 63.5 mm to (165.3, 81.4)
- moved U2 59.2 mm to (161.1, 78.8), turned to 90 degrees
- moved C5 57.8 mm to (164.3, 85.7), turned to 270 degrees
- moved U3 57.0 mm to (161.1, 82.5), turned to 90 degrees
- moved C11 49.6 mm to (154.5, 85.7), turned to 90 degrees
- moved R2 46.5 mm to (158.0, 84.8), turned to 90 degrees
- moved R3 45.0 mm to (152.1, 84.8), turned to 0 degrees
- moved J1 42.8 mm to (121.7, 67.0)
- moved R1 39.0 mm to (161.2, 70.5)
- moved C6 38.8 mm to (163.2, 72.2), turned to 90 degrees
- moved U4 38.5 mm to (151.4, 79.9), turned to 0 degrees
- moved C9 36.2 mm to (155.9, 78.0)
- moved C8 32.9 mm to (146.8, 84.8), turned to 270 degrees
- moved C10 32.8 mm to (147.3, 74.2)
- moved C12 31.3 mm to (145.3, 80.9), turned to 270 degrees
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Connections:
- J1 pad B2: Net-(J1-PadB2) -> JTAG_TRST
- J1 pad B3: Net-(J1-PadB3) -> JTAG_TDI
- J1 pad B4: Net-(J1-PadB4) -> JTAG_TDO
- J1 pad B5: Net-(J1-PadB5) -> JTAG_TMS
- J1 pad B6: Net-(J1-PadB6) -> JTAG_TCK
- U4 pad 10: XTAL_XO -> Net-(U4-Pad10)
- U4 pad 38: RX -> GPIO1
- U4 pad 39: TX -> GPIO2
- U4 pad 9: XTAL_XI -> CLKIN
Routing:
- net +3V3: track 23.9 -> 110.4 mm, vias 0 -> 5
- net LED2: track 0.00 -> 61.4 mm, vias 0 -> 2
- net LED1: track 0.00 -> 55.2 mm, vias 0 -> 2
- net JTAG_TRST: track 3.44 -> 55.2 mm, vias 0 -> 2
- net VCC_CLEAN: track 4.88 -> 54.0 mm, vias 0 -> 4
- net UFO.RST: track 0.00 -> 46.9 mm, vias 0 -> 1
- net GPIO2: track 0.00 -> 46.7 mm, vias 0 -> 1
- net GPIO1: track 0.00 -> 45.9 mm, vias 0 -> 1
- net GPIO4: track 0.00 -> 45.8 mm, vias 0 -> 2
- net FTDI.JTAG_TCK: track 45.4 -> 0.00 mm
- net CLKIN: track 0.00 -> 39.8 mm
- net FTDI.JTAG_TDI: track 38.6 -> 0.00 mm
- net FTDI.JTAG_TDO: track 35.2 -> 0.00 mm
- net FTDI.JTAG_TMS: track 32.4 -> 0.00 mm
- net Net-(C7-Pad1): track 3.95 -> 32.2 mm, vias 0 -> 2
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- added copper zone on B.Cu, net GND
- added copper zone on F.Cu, net GND
Other:
- board size 53.3 x 67.3 mm -> 54 x 65 mm
- net class Default: clearance 0.127 -> 0.12
- rule pad_to_mask_clearance: 0.051 -> 0
- rule trace_clearance: 0.127 -> 0.12
- rule trace_min: 0.0889 -> 0.2
- rule via_min_drill: 0.2 -> 0.3
- rule via_min_size: 0.45 -> 0.4

Commit message: revision 0.1
Parts:
- removed SW1: SW_Push, Button_Switch_SMD:SW_SPST_B3U-1000P
- added G***: LOGO, cw308_fe310:logo, B.Cu at (155.2, 107.5)
- added J2: SerialSel, Connector_PinHeader_2.54mm:PinHeader_2x02_P2.54mm_Vertical, F.Cu at (125.5, 67.5)
- C1, C10, C11, C12, C13, C4, C5, C6, C7, C8, C9: footprint Capacitor_SMD:C_0603_1608Metric_Pad1.05x0.95mm_HandSolder -> Capacitor_SMD:C_0603_1608Metric
- R1, R2, R3, R4: footprint Resistor_SMD:R_0603_1608Metric_Pad1.05x0.95mm_HandSolder -> Resistor_SMD:R_0603_1608Metric
- moved C10 0.21 mm to (147.5, 74.2)
Connections:
- J1 pad C20: LED2 -> LED3
- U4 pad 38: GPIO1 -> RX
- U4 pad 39: GPIO2 -> TX
- U4 pad 43: LED2 -> LED3
Routing:
- net LED3: track 0.00 -> 60.0 mm, vias 0 -> 1
- net RX: track 0.00 -> 34.5 mm, vias 0 -> 1
- net TX: track 0.00 -> 30.0 mm, vias 0 -> 1
- net GPIO2: track 46.7 -> 16.8 mm, vias 1 -> 0
- net GPIO1: track 45.9 -> 16.4 mm, vias 1 -> 0
- net Net-(C7-Pad1): track 32.2 -> 13.7 mm, vias 2 -> 0
- net +1V8: track 48.7 -> 61.8 mm
- net FLASH_IO0: track 12.4 -> 21.0 mm
- net Net-(C6-Pad2): track 9.07 -> 16.8 mm
- net FLASH_SCK: track 14.5 -> 21.0 mm
- net FLASH_IO3: track 16.2 -> 21.0 mm
- net FLASH_IO2: track 16.6 -> 21.2 mm
- net GPIO4: track 45.8 -> 44.0 mm
- net +3V3: track 110.4 -> 109.0 mm
- net LED2: track 61.4 -> 62.8 mm
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Other:
- board size 54 x 65 mm -> 56 x 67 mm
- board text added: "1V8"
- board text added: "3V3"
- board text added: "CLK"
- board text added: "FE310 Target Board For ChipWhisperer CW308 UFO Board"
- board text added: "R"
- board text added: "Rev 0.1"
- board text added: "SHUNT"
- board text added: "T"
- board text added: "X"
- board text added: "https://adamws.xyz"
